File: sniffer.kicad_pcb (KiCad board)
At the start: 2 copper layers, 30 x 61.6 mm, 45 parts, among them J1 TRACK, J2 TRACK, Q1 BC857B, Q2 BC857B, Q3 BC857B, Q4 BC857B, U1 LM393, U2 TL431A, U3 SLHT50H, U4 HCPL2630SDM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

Commit message: fix: U3 regulator pins flipped (#1)
Parts:
- moved U3 1.10 mm to (149.1, 128.9), turned to 180 degrees
Connections:
- U3 pad 2: +VT -> +5VP
- U3 pad 3: +5VP -> +VT
Routing:
- net P: track 0.00 -> 6.11 mm
- net +VT: track 17.3 -> 19.2 mm
- net P1: track 18.7 -> 20.2 mm
- net +5VP: track 56.9 -> 55.5 mm
Other:
- board text added: "0.1.1"
- board text removed: "0.1.0"

Commit message: chore: suitable names for `BIDI_DATA` and `BIDI_POL`
Connections:
- net BIDI_DATA renamed BIDI_P
- net BIDI_POL renamed BIDI_N
Changed lines of the file:
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@@
 			(layers "F.Cu" "F.Mask" "F.Paste")
 			(roundrect_rratio 0.25)
-			(net "BIDI_DATA")
+			(net "BIDI_P")
 			(pintype "open_collector")
 		)
@@
 			(layers "F.Cu" "F.Mask" "F.Paste")
 			(roundrect_rratio 0.25)
-			(net "BIDI_POL")
+			(net "BIDI_N")
 			(pintype "open_collector")
 		)
@@
 			(layers "F.Cu" "F.Mask" "F.Paste")
 			(roundrect_rratio 0.25)
-			(net "BIDI_POL")
+			(net "BIDI_N")
 			(pinfunction "B_1")
 			(pintype "input")
@@
 			(layers "F.Cu" "F.Mask" "F.Paste")
 			(roundrect_rratio 0.208333)
-			(net "BIDI_DATA")
+			(net "BIDI_P")
 			(pintype "passive")
 		)
@@
 			(layers "F.Cu" "F.Mask" "F.Paste")
 			(roundrect_rratio 0.25)
-			(net "BIDI_DATA")
+			(net "BIDI_P")
 			(pinfunction "B_1")
 			(pintype "input")
@@
 			(layers "F.Cu" "F.Mask" "F.Paste")
 			(roundrect_rratio 0.208333)
-			(net "BIDI_POL")
+			(net "BIDI_N")
 			(pintype "passive")
 		)
@@
 			(layers "F.Cu" "F.Mask" "F.Paste")
 			(roundrect_rratio 0.25)
-			(net "BIDI_POL")
+			(net "BIDI_N")
 			(pinfunction "B_1")
 			(pintype "input")
@@
 	)
 	(segment
-		(start 149.9 117.359412)
-		(end 149.9 115.15)
-		(width 0.2)
-		(layer "F.Cu")
-		(net "BIDI_DATA")
-	)
-	(segment
-		(start 150.905 118.925)
-		(end 152.325 118.925)
-		(width 0.2)
-		(layer "F.Cu")
-		(net "BIDI_DATA")
-	)
-	(segment
-		(start 149.9 115.15)
-		(end 151.55 113.5)
-		(width 0.2)
-		(layer "F.Cu")
-		(net "BIDI_DATA")
-	)
-	(segment
-		(start 150.905 118.364412)
-		(end 149.9 117.359412)
-		(width 0.2)
-		(layer "F.Cu")
-		(net "BIDI_DATA")
-	)
-	(segment
 		(start 147.095 126.004412)
 		(end 147.095 123.875)
@@
 	)
 	(segment
-		(start 154.3 118)
-		(end 154.9 118)
-		(width 0.2)
-		(layer "F.Cu")
-		(net "BIDI_POL")
-	)
-	(segment
-		(start 149.635 123.875)
-		(end 149.635 122.900001)
-		(width 0.2)
-		(layer "F.Cu")
-		(net "BIDI_POL")
-	)
-	(segment
-		(start 157.373 114.677)
-		(end 156.227 114.677)
-		(width 0.2)
-		(layer "F.Cu")
-		(net "BIDI_POL")
-	)
-	(segment
-		(start 151.435001 121.1)
-		(end 152.6 121.1)
-		(width 0.2)
-		(layer "F.Cu")
-		(net "BIDI_POL")
-	)
-	(segment
-		(start 155.05 114.95)
-		(end 155 115)
-		(width 0.2)
-		(layer "F.Cu")
-		(net "BIDI_POL")
-	)
-	(segment
-		(start 153.6 120.1)
-		(end 153.6 118.7)
-		(width 0.2)
-		(layer "F.Cu")
-		(net "BIDI_POL")
-	)
-	(segment
-		(start 155.05 113.5)
-		(end 155.05 114.95)
-		(width 0.2)
-		(layer "F.Cu")
-		(net "BIDI_POL")
-	)
-	(segment
-		(start 149.635 122.900001)
-		(end 151.435001 121.1)
-		(width 0.2)
-		(layer "F.Cu")
-		(net "BIDI_POL")
-	)
-	(segment
-		(start 152.6 121.1)
-		(end 153.6 120.1)
-		(width 0.2)
-		(layer "F.Cu")
-		(net "BIDI_POL")
-	)
-	(segment
-		(start 153.6 118.7)
-		(end 154.3 118)
-		(width 0.2)
-		(layer "F.Cu")
-		(net "BIDI_POL")
-	)
-	(segment
-		(start 158.55 113.5)
-		(end 157.373 114.677)
-		(width 0.2)
-		(layer "F.Cu")
-		(net "BIDI_POL")
-	)
-	(segment
-		(start 156.227 114.677)
-		(end 155.05 113.5)
-		(width 0.2)
-		(layer "F.Cu")
-		(net "BIDI_POL")
-	)
-	(via
-		(at 155 115)
-		(size 0.6)
-		(drill 0.3)
-		(layers "F.Cu" "B.Cu")
-		(net "BIDI_POL")
-	)
-	(via
-		(at 154.9 118)
-		(size 0.6)
-		(drill 0.3)
-		(layers "F.Cu" "B.Cu")
-		(net "BIDI_POL")
-	)
-	(segment
-		(start 155 117.9)
-		(end 154.9 118)
-		(width 0.2)
-		(layer "B.Cu")
-		(net "BIDI_POL")
-	)
-	(segment
-		(start 155 115)
-		(end 155 117.9)
-		(width 0.2)
-		(layer "B.Cu")
-		(net "BIDI_POL")
-	)
-	(segment
 		(start 140.5 129.3)
 		(end 141.1 129.9)
@@
 		(net "Net-(A1-GPIO0)")
 	)
+	(segment
+		(start 149.9 117.359412)
+		(end 149.9 115.15)
+		(width 0.2)
+		(layer "F.Cu")
+		(net "BIDI_P")
+	)
+	(segment
+		(start 150.905 118.925)
+		(end 152.325 118.925)
+		(width 0.2)
+		(layer "F.Cu")
+		(net "BIDI_P")
+	)
+	(segment
+		(start 149.9 115.15)
+		(end 151.55 113.5)
+		(width 0.2)
+		(layer "F.Cu")
+		(net "BIDI_P")
+	)
+	(segment
+		(start 150.905 118.364412)
+		(end 149.9 117.359412)
+		(width 0.2)
+		(layer "F.Cu")
+		(net "BIDI_P")
+	)
+	(segment
+		(start 154.3 118)
+		(end 154.9 118)
+		(width 0.2)
+		(layer "F.Cu")
+		(net "BIDI_N")
+	)
+	(segment
+		(start 149.635 123.875)
+		(end 149.635 122.900001)
+		(width 0.2)
+		(layer "F.Cu")
+		(net "BIDI_N")
+	)
+	(segment
+		(start 157.373 114.677)
+		(end 156.227 114.677)
+		(width 0.2)
+		(layer "F.Cu")
+		(net "BIDI_N")
+	)
+	(segment
+		(start 151.435001 121.1)
+		(end 152.6 121.1)
+		(width 0.2)
+		(layer "F.Cu")
+		(net "BIDI_N")
+	)
+	(segment
+		(start 155.05 114.95)
+		(end 155 115)
+		(width 0.2)
+		(layer "F.Cu")
+		(net "BIDI_N")
+	)
+	(segment
+		(start 153.6 120.1)
+		(end 153.6 118.7)
+		(width 0.2)
+		(layer "F.Cu")
+		(net "BIDI_N")
+	)
+	(segment
+		(start 155.05 113.5)
+		(end 155.05 114.95)
+		(width 0.2)
+		(layer "F.Cu")
+		(net "BIDI_N")
+	)
+	(segment
+		(start 149.635 122.900001)
+		(end 151.435001 121.1)
+		(width 0.2)
+		(layer "F.Cu")
+		(net "BIDI_N")
+	)
+	(segment
+		(start 152.6 121.1)
+		(end 153.6 120.1)
+		(width 0.2)
+		(layer "F.Cu")
+		(net "BIDI_N")
+	)
+	(segment
+		(start 153.6 118.7)
+		(end 154.3 118)
+		(width 0.2)
+		(layer "F.Cu")
+		(net "BIDI_N")
+	)
+	(segment
+		(start 158.55 113.5)
+		(end 157.373 114.677)
+		(width 0.2)
+		(layer "F.Cu")
+		(net "BIDI_N")
+	)
+	(segment
+		(start 156.227 114.677)
+		(end 155.05 113.5)
+		(width 0.2)
+		(layer "F.Cu")
+		(net "BIDI_N")
+	)
+	(via
+		(at 155 115)
+		(size 0.6)
+		(drill 0.3)
+		(layers "F.Cu" "B.Cu")
+		(net "BIDI_N")
+	)
+	(via
+		(at 154.9 118)
+		(size 0.6)
+		(drill 0.3)
+		(layers "F.Cu" "B.Cu")
+		(net "BIDI_N")
+	)
+	(segment
+		(start 155 117.9)
+		(end 154.9 118)
+		(width 0.2)
+		(layer "B.Cu")
+		(net "BIDI_N")
+	)
+	(segment
+		(start 155 115)
+		(end 155 117.9)
+		(width 0.2)
+		(layer "B.Cu")
+		(net "BIDI_N")
+	)
 	(zone
